File: kicad/SerialtoHID.kicad_pcb (KiCad board)
At the start: 0 parts

Commit message: a
Parts:
- added C1: 22pF, Capacitor_SMD:C_0603_1608Metric, F.Cu at (114.3, 101.6)
- added C2: 22pF, Capacitor_SMD:C_0603_1608Metric, F.Cu at (90.6, 108.9)
- added C3: 1uF, Capacitor_SMD:C_0603_1608Metric, F.Cu at (90.6, 106.3)
- added C4: 0.1uF, Capacitor_SMD:C_0603_1608Metric, F.Cu at (86.6, 106.3)
- added J1: USB_B, Connector_USB:USB_Micro-B_Wuerth_629105150521, F.Cu at (67.0, 113.1)
- added J2: DB9_Male_MountingHoles, Connector_Dsub:DSUB-9_Male_Horizontal_P2.77x2.84mm_EdgePinOffset7.70mm_Housed_MountingHolesOffset9.12mm, F.Cu at (90.3, 87.1)
- added R1: 10k, Resistor_SMD:R_0603_1608Metric, F.Cu at (125.2, 85.1)
- added R2: 10k, Resistor_SMD:R_0603_1608Metric, F.Cu at (86.6, 108.9)
- added U1: ATmega32U2-M, Package_DFN_QFN:QFN-32-1EP_5x5mm_P0.5mm_EP3.1x3.1mm, F.Cu at (90.5, 96.7)
- added Y1: 16MHz, Crystal:Crystal_SMD_3225-4Pin_3.2x2.5mm, F.Cu at (82.0, 107.3)
Other:
- copper layers 0 -> 2
