File: kicad/SerialtoHID.kicad_sch (KiCad schematic)
At the start: 10 parts

Commit message: a
Parts:
- added C5, C6: 0.1uF, Capacitor_SMD:C_0603_1608Metric, symbol Device:C
- added C7, C8, C9: 0.47uF, Capacitor_SMD:C_0603_1608Metric, symbol Device:C
- added U2: MAX3232, Package_SO:SOIC-16_3.9x9.9mm_P1.27mm, symbol Interface_UART:MAX3232
- C1, C2, C3, C4: renamed from C?; footprint (none) -> Capacitor_SMD:C_0603_1608Metric
- J1: renamed from J?; footprint (none) -> Connector_USB:USB_Micro-B_Wuerth_629105150521
- J2: renamed from J?; footprint (none) -> Connector_Dsub:DSUB-9_Male_Horizontal_P2.77x2.84mm_EdgePinOffset7.70mm_Housed_MountingHolesOffset9.12mm
- R1, R2: renamed from R?; footprint (none) -> Resistor_SMD:R_0603_1608Metric
- Y1: renamed from Y?; footprint (none) -> Crystal:Crystal_SMD_3225-4Pin_3.2x2.5mm
- gave numbers to parts that had none: 1
Connections:
- net GND: now also C6.2, C9.2, U2.15 (GND)
- net MOUSE_TX: now also U2.13 (R1IN); no longer R2.1, U1.8 (PD2)
- net VCC: now also C6.1, C8.2, U2.16 (VCC)
- net TTL_RX: now reaches U1.6 (PD0)
- net TTL_RX: now also U2.11 (T1IN)
- net TTL_TX: now reaches U1.7 (PD1)
- net TTL_TX: now also U2.12 (R1OUT)
- net MOUSE_RX: now reaches J2.2
- net MOUSE_RX: now also U2.14 (T1OUT)
- new net: R2.1, U1.8 (PD2)
- new net: C9.1, U2.6 (VS-)
- new net: C7.1, U2.4 (C2+)
- new net: C7.2, U2.5 (C2-)
- new net: C5.1, U2.1 (C1+)
- new net: C5.2, U2.3 (C1-)
- new net: C8.1, U2.2 (VS+)
- no-connect marks 6 -> 5
